File: half-bridge.kicad_pcb (KiCad board)
At the start: 2 copper layers, 38.1 x 24.1 mm, 19 parts, among them P1 CONN_01X04, P2 CONN_01X02, P3 CONN_01X02, P4 CONN_01X03, Q1 Q_NMOS_GDS, Q2 Q_NMOS_GDS, U1 MOSFET_DRIVER_FAN7842MX

Commit message: Added output sense circuit
Parts:
- P1: value CONN_01X04 -> CONN_01X05; footprint lib_pcb:CON_1x4_0.1in -> lib_pcb:CON_1x5_0.1in
- P2, P3: value CONN_01X02 -> CONN_01X04; footprint lib_pcb:CON_1x2_0.1in -> lib_pcb:CON_1x4_0.1in
- moved C4 5.34 mm to (170.2, 63.2)
- moved P2 2.29 mm to (175.3, 66.3)
- moved P3 1.98 mm to (172.7, 66.3), turned to 270 degrees
- moved P1 1.52 mm to (165.1, 70.1)
Connections:
- C1 pad 2: Net-(C1-Pad2) -> /Vout
- P1 pad 4: GND -> /Vout
- P2 pad 2: +12V -> +BATT
- P3 pad 1: +BATT -> GND
- P4 pad 1: Net-(C1-Pad2) -> /Vout
- Q1 pad 3: Net-(C1-Pad2) -> /Vout
- Q2 pad 2: Net-(C1-Pad2) -> /Vout
- R1 pad 2: Net-(C1-Pad2) -> /Vout
- R3 pad 2: Net-(C1-Pad2) -> /Vout
- R4 pad 1: Net-(C1-Pad2) -> /Vout
- U1 pad 6: Net-(C1-Pad2) -> /Vout
Routing:
- net /Vout: track 0.00 -> 21.6 mm, vias 0 -> 1
- net Net-(C1-Pad2): track 10.0 -> 0.00 mm
- net GND: track 14.0 -> 4.37 mm
- added copper zone on F.Cu, net /Vout
- added copper zone on F.Cu, net GND
- removed copper zone on F.Cu, net Net-(C1-Pad2)
Other:
- rule pad_to_mask_clearance: 0.2 -> 0.0508
- board text added: "FB"
- board text added: "G"
- board text removed: "GND"
